File: Kicad File/Arduino Mini.kicad_pcb (KiCad board)
At the start: 2 copper layers, 21 x 21 mm, 2 parts, among them U1 ATmega328P-A, Y1 Crystal_GND3_Small

Commit message: add Gerber
Parts:
- added C1: 0.1uF, Capacitor_SMD:C_0805_2012Metric, F.Cu at (152.1, 96.9)
- added C2: 0.1uF, Capacitor_SMD:C_0805_2012Metric, F.Cu at (141.9, 96.9)
- added C3: 100nF, Capacitor_SMD:C_0805_2012Metric, B.Cu at (146.0, 102.0)
- added C4: 100nF, Capacitor_SMD:C_0805_2012Metric, B.Cu at (148.0, 102.0)
- added C5: 100nF, Capacitor_SMD:C_0805_2012Metric, B.Cu at (150.1, 102.0)
- added D1: 1N5819WS, Diode_SMD:D_SOD-323, B.Cu at (144.0, 102.0)
- added J1: Conn_01x08_Pin, Connector_PinHeader_2.54mm:PinHeader_1x08_P2.54mm_Vertical, B.Cu at (155.9, 93.1)
- added J2: Conn_01x08_Pin, Connector_PinHeader_2.54mm:PinHeader_1x08_P2.54mm_Vertical, B.Cu at (138.1, 110.9)
- added J3: Conn_01x06_Pin, Connector_PinHeader_2.54mm:PinHeader_1x06_P2.54mm_Vertical, B.Cu at (138.1, 95.7)
- added J4: Conn_01x06_Pin, Connector_PinHeader_2.54mm:PinHeader_1x06_P2.54mm_Vertical, B.Cu at (155.9, 108.3)
- added R1: R, Resistor_SMD:R_0805_2012Metric, B.Cu at (147.0, 96.9)
- added S1: EVPBB4A9B000, EVPBB4A9B000:SW_EVPBB4A9B000, F.Cu at (152.1, 107.1)
- moved Y1 0.61 mm to (141.9, 107.1)
Connections:
- U1 pad 1: unconnected-(U1-PD3-Pad1) -> /D3
- U1 pad 10: unconnected-(U1-PD6-Pad10) -> /D6
- U1 pad 11: unconnected-(U1-PD7-Pad11) -> /D7
- U1 pad 12: unconnected-(U1-PB0-Pad12) -> /D8
- U1 pad 13: unconnected-(U1-PB1-Pad13) -> /D9
- U1 pad 14: unconnected-(U1-PB2-Pad14) -> /D10
- U1 pad 15: unconnected-(U1-PB3-Pad15) -> /MOSI
- U1 pad 16: unconnected-(U1-PB4-Pad16) -> /MISO
- U1 pad 17: unconnected-(U1-PB5-Pad17) -> /SCK
- U1 pad 18: unconnected-(U1-AVCC-Pad18) -> VCC
- U1 pad 19: unconnected-(U1-ADC6-Pad19) -> /A6
- U1 pad 2: unconnected-(U1-PD4-Pad2) -> /D4
- U1 pad 20: unconnected-(U1-AREF-Pad20) -> Net-(U1-AREF)
- U1 pad 21: Net-(U1-GND-Pad21) -> GND
- U1 pad 22: unconnected-(U1-ADC7-Pad22) -> /A7
- U1 pad 23: unconnected-(U1-PC0-Pad23) -> /A0
- U1 pad 24: unconnected-(U1-PC1-Pad24) -> /A1
- U1 pad 25: unconnected-(U1-PC2-Pad25) -> /A2
- U1 pad 26: unconnected-(U1-PC3-Pad26) -> /A3
- U1 pad 27: unconnected-(U1-PC4-Pad27) -> /A4
- U1 pad 28: unconnected-(U1-PC5-Pad28) -> /A5
- U1 pad 29: unconnected-(U1-~{RESET}/PC6-Pad29) -> /RESET
- U1 pad 3: Net-(U1-GND-Pad21) -> GND
- U1 pad 30: unconnected-(U1-PD0-Pad30) -> /RX
- U1 pad 31: unconnected-(U1-PD1-Pad31) -> /TX
- U1 pad 32: unconnected-(U1-PD2-Pad32) -> /D2
- U1 pad 4: Net-(U1-VCC-Pad4) -> VCC
- U1 pad 5: Net-(U1-GND-Pad21) -> GND
- U1 pad 6: Net-(U1-VCC-Pad4) -> VCC
- U1 pad 7: unconnected-(U1-XTAL1/PB6-Pad7) -> Net-(U1-XTAL1/PB6)
- U1 pad 8: unconnected-(U1-XTAL2/PB7-Pad8) -> Net-(U1-XTAL2/PB7)
- U1 pad 9: unconnected-(U1-PD5-Pad9) -> /D5
- Y1 pad 1: unconnected-(Y1-Pad1) -> Net-(U1-XTAL2/PB7)
- Y1 pad 2: unconnected-(Y1-Pad2) -> Net-(U1-XTAL1/PB6)
- Y1 pad 3: unconnected-(Y1-Pad3) -> GND
Routing:
- net /RESET: track 0.00 -> 33.7 mm, vias 0 -> 6
- net VCC: track 0.00 -> 22.6 mm, vias 0 -> 2
- net /A6: track 0.00 -> 18.0 mm, vias 0 -> 1
- net /D2: track 0.00 -> 11.6 mm
- net /D3: track 0.00 -> 9.67 mm, vias 0 -> 1
- net /D4: track 0.00 -> 9.52 mm, vias 0 -> 1
- net /D8: track 0.00 -> 8.49 mm
- net /A7: track 0.00 -> 7.77 mm, vias 0 -> 1
- net /D7: track 0.00 -> 7.36 mm
- net /A5: track 0.00 -> 7.11 mm, vias 0 -> 1
- net /D9: track 0.00 -> 7.10 mm
- net /A0: track 0.00 -> 6.61 mm
- net /RX: track 0.00 -> 6.25 mm, vias 0 -> 1
- net +5V: track 0.00 -> 5.93 mm
- net Net-(U1-XTAL1/PB6): track 0.00 -> 5.89 mm, vias 0 -> 2
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- added copper zone on B.Cu, net GND
- added copper zone on F.Cu, net GND
