File: Kicad File/Arduino Mini.kicad_sch (KiCad schematic)
At the start: 1 part, among them U1 ATmega328P-A

Commit message: update pcb
Parts:
- added Y1: Crystal_GND3_Small, Crystal:Resonator_SMD_Murata_CSTxExxV-3Pin_3.0x1.1mm, symbol Device:Crystal_GND3_Small
Other:
- company: (none) -> Zhejiang University
- title: (none) -> Arduino Mini
Changed lines of the file:
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@@
 (kicad_sch (version 20230121) (generator eeschema)
   (paper "A4")
+  (title_block
+    (title "Arduino Mini")
+    (date "2023-10-18")
+    (rev "V0.2")
+    (company "Zhejiang University")
+    (comment 1 "DTB Lab")
+    (comment 4 "Xin An")
+  )
+  (symbol (lib_id "Device:Crystal_GND3_Small") (at 133.604 122.936 0) (unit 1)
+    (in_bom yes) (on_board yes) (dnp no) (fields_autoplaced)
+    (property "Reference" "Y1" (at 133.604 116.84 0)
+      (effects (font (size 1.27 1.27)))
+    )
+    (property "Value" "Crystal_GND3_Small" (at 133.604 119.38 0)
+      (effects (font (size 1.27 1.27)))
+    )
+    (property "Footprint" "Crystal:Resonator_SMD_Murata_CSTxExxV-3Pin_3.0x1.1mm" (at 133.604 122.936 0)
+      (effects (font (size 1.27 1.27)) hide)
+    )
+    (property "Datasheet" "~" (at 133.604 122.936 0)
+      (effects (font (size 1.27 1.27)) hide)
+    )
+    (pin "1")
+    (pin "2")
+    (pin "3")
+    (instances
+      (project "Arduino Mini"
+        (path "/542141a7-426a-4277-866a-9b4fbf779468"
+          (reference "Y1") (unit 1)
+        )
+      )
+    )
+  )
   (symbol (lib_id "MCU_Microchip_ATmega:ATmega328P-A") (at 70.104 108.204 0) (unit 1)
     (in_bom yes) (on_board yes) (dnp no) (fields_autoplaced)

Commit message: add Gerber
Parts:
- added C1, C2: 0.1uF, Capacitor_SMD:C_0805_2012Metric, symbol Device:C
- added C3, C4, C5: 100nF, Capacitor_SMD:C_0805_2012Metric, symbol Device:C
- added D1: 1N5819WS, Diode_SMD:D_SOD-323, symbol Diode:1N5819WS
- added J1, J2: Conn_01x08_Pin, Connector_PinHeader_2.54mm:PinHeader_1x08_P2.54mm_Vertical, symbol Connector:Conn_01x08_Pin
- added J3, J4: Conn_01x06_Pin, Connector_PinHeader_2.54mm:PinHeader_1x06_P2.54mm_Vertical, symbol Connector:Conn_01x06_Pin
- added R1: R, Resistor_SMD:R_0805_2012Metric, symbol Device:R
- added S1: EVPBB4A9B000, EVPBB4A9B000:SW_EVPBB4A9B000, symbol EVPBB4A9B000:EVPBB4A9B000
Connections:
- net at Y1.1: now also U1.8 (XTAL2/PB7)
- net at Y1.2: now also U1.7 (XTAL1/PB6)
- net GND: now reaches Y1.3
- net GND: now also U1.21 (GND), U1.3 (GND), U1.5 (GND), C1.1, C3.2, C4.2, C5.2, J1.1 (Pin_1), J2.1 (Pin_1), J3.5 (Pin_5), S1.B2
- net D3: now reaches U1.1 (PD3)
- net D3: now also J2.3 (Pin_3)
- net D6: now reaches U1.10 (PD6)
- net D6: now also J2.6 (Pin_6)
- net D7: now reaches U1.11 (PD7)
- net D7: now also J2.7 (Pin_7)
- net D8: now reaches U1.12 (PB0)
- net D8: now also J2.8 (Pin_8)
- net D9: now reaches U1.13 (PB1)
- net D9: now also J4.1 (Pin_1)
- net D10: now reaches U1.14 (PB2)
- net D10: now also J4.2 (Pin_2)
- net MOSI: now reaches U1.15 (PB3)
- net MOSI: now also J4.3 (Pin_3)
- net MISO: now reaches U1.16 (PB4)
- net MISO: now also J4.4 (Pin_4)
- net SCK: now reaches U1.17 (PB5)
- net SCK: now also J4.5 (Pin_5)
- net VCC: now reaches U1.18 (AVCC)
- net VCC: now also U1.4 (VCC), U1.6 (VCC), C3.1, C4.1, C5.1, D1.1 (K), R1.2
- net A6: now reaches U1.19 (ADC6)
- net A6: now also J1.8 (Pin_8)
- net D4: now reaches U1.2 (PD4)
- net D4: now also J2.4 (Pin_4)
- net at U1.20 (AREF): now also C1.2
- net A7: now reaches U1.22 (ADC7)
- net A7: now also J4.6 (Pin_6)
- net A0: now reaches U1.23 (PC0)
- net A0: now also J1.2 (Pin_2)
- net A1: now reaches U1.24 (PC1)
- net A1: now also J1.3 (Pin_3)
- net A2: now reaches U1.25 (PC2)
- net A2: now also J1.4 (Pin_4)
- net A3: now reaches U1.26 (PC3)
- net A3: now also J1.5 (Pin_5)
- net A4: now reaches U1.27 (PC4)
- net A4: now also J1.6 (Pin_6)
- net A5: now reaches U1.28 (PC5)
- net A5: now also J1.7 (Pin_7)
- net RESET: now reaches U1.29 (~{RESET}/PC6)
- net RESET: now also C2.1, J3.6 (Pin_6), R1.1, S1.A1
- net RX: now reaches U1.30 (PD0)
- net RX: now also J3.3 (Pin_3)
- net TX: now reaches U1.31 (PD1)
- net TX: now also J3.2 (Pin_2)
- net D2: now reaches U1.32 (PD2)
- net D2: now also J2.2 (Pin_2)
- net D5: now reaches U1.9 (PD5)
- net D5: now also J2.5 (Pin_5)
- new net +5V: D1.2 (A), J3.4 (Pin_4)
- new net DTR: C2.2, J3.1 (Pin_1)
Other:
- moved on the sheet: U1, Y1
